File: backlight_circuit_boards/center_gauges/center_gauges_backlight.kicad_pcb (KiCad board)
At the start: 2 copper layers, 84.7 x 28 mm, 10 parts, among them J1 IN, J2 OUT

Commit message: improvements to all boards
Parts:
- added C5: 10 uF, Capacitors_Tantalum_SMD:CP_Tantalum_Case-D_EIA-7343-31_Reflow, F.Cu at (55.0, 33.6)
- D1, D2, D3, D4: footprint LEDs:LED_WS2812B-PLCC4 -> Sparkfun LEDs:LED_WS2812B-PLCC4_HandSoldering
- J1, J2: footprint Pin_Headers:Pin_Header_Straight_1x03_Pitch2.54mm -> Frickelbude Connectors:wire_solder_pads_1x03_2.5x1.7mm_Pitch2.54mm; moved to F.Cu
- moved J2 27.4 mm to (117.3, 48.9), turned to 345 degrees
- moved J1 27.4 mm to (43.3, 48.8), turned to 15 degrees
- moved D1 19.4 mm to (47.9, 41.6), turned to 225 degrees
- moved D3 19.3 mm to (91.9, 41.6), turned to 225 degrees
- moved D4 19.3 mm to (112.4, 41.6), turned to 135 degrees
- moved D2 19.2 mm to (68.4, 41.6), turned to 135 degrees
- moved C3 2.14 mm to (116.8, 37.4), turned to 135 degrees
- moved C2 1.39 mm to (43.8, 37.3)
- moved C1 1.25 mm to (73.4, 36.6), turned to 135 degrees
- moved C4 1.13 mm to (87.2, 36.5), turned to 225 degrees
Routing:
- net Net-(D2-Pad2): track 86.0 -> 22.0 mm
- net VDD: track 114.2 -> 156.5 mm
- net GND: track 10.3 -> 0.00 mm
- net Net-(D4-Pad2): track 9.25 -> 12.9 mm
- net Net-(D3-Pad2): track 16.4 -> 19.7 mm
- net Net-(D1-Pad2): track 17.2 -> 19.2 mm
- net Net-(D1-Pad4): track 10.7 -> 9.06 mm
Other:
- board size 84.7 x 28 mm -> 84.7 x 28.1 mm
